File: Python/KicadPyBentley/pcb/pcbs/V5/V5.kicad_pcb (KiCad board)
At the start: 4 copper layers, 470.8 x 1453.1 mm, 192 parts

Commit message: solved footprints bug
Parts:
- removed the REF** at (122.7, 352.8)
- removed the REF** at (15.9, 84.9)
- removed the REF** at (26.7, 84.4)
- removed the REF** at (37.6, 83.9)
- removed the REF** at (48.4, 83.4)
- removed the REF** at (59.3, 82.9)
- removed the REF** at (72.2, 82.4)
- removed the REF** at (81.8, 82.0)
- removed the REF** at (91.4, 81.7)
- removed the REF** at (101.0, 81.4)
- removed the REF** at (110.6, 81.0)
- removed the REF** at (133.8, 393.6)
- removed the REF** at (120.1, 80.7)
- removed the REF** at (129.7, 80.4)
- removed the REF** at (142.5, 80.0)
- removed the REF** at (153.2, 79.7)
- removed the REF** at (163.9, 79.4)
- removed the REF** at (174.6, 79.1)
- removed the REF** at (185.2, 78.9)
- removed the REF** at (195.9, 78.6)
- removed the REF** at (208.6, 78.3)
- removed the REF** at (219.2, 78.0)
- removed the REF** at (144.1, 434.6)
- removed the REF** at (229.7, 77.8)
- removed the REF** at (240.3, 77.6)
- removed the REF** at (250.8, 77.3)
- removed the REF** at (261.3, 77.1)
- removed the REF** at (274.0, 76.9)
- removed the REF** at (282.9, 76.7)
- removed the REF** at (291.8, 76.5)
- removed the REF** at (300.7, 76.3)
- removed the REF** at (309.7, 76.1)
- removed the REF** at (318.6, 75.9)
- removed the REF** at (150.7, 478.3)
- removed the REF** at (331.1, 75.7)
- removed the REF** at (340.5, 75.5)
- removed the REF** at (349.8, 75.3)
- removed the REF** at (359.1, 75.1)
- removed the REF** at (368.4, 74.9)
- removed the REF** at (380.9, 74.7)
- removed the REF** at (390.6, 74.4)
- removed the REF** at (400.2, 74.5)
- removed the REF** at (409.8, 74.9)
- removed the REF** at (419.5, 75.4)
- removed the REF** at (149.3, 520.7)
- removed the REF** at (432.1, 76.5)
- removed the REF** at (442.0, 77.7)
- removed the REF** at (451.9, 79.2)
- removed the REF** at (461.9, 81.2)
- removed the REF** at (474.8, 84.3)
- removed the REF** at (483.4, 86.9)
- removed the REF** at (492.1, 89.9)
- removed the REF** at (500.8, 92.9)
- removed the REF** at (513.7, 97.5)
- removed the REF** at (522.5, 99.0)
- removed the REF** at (150.4, 554.6)
- removed the REF** at (531.3, 99.1)
- removed the REF** at (540.0, 99.2)
- removed the REF** at (552.9, 81.9)
- removed the REF** at (562.4, 66.3)
- removed the REF** at (571.0, 55.8)
- removed the REF** at (578.9, 49.5)
- removed the REF** at (588.3, 43.9)
- removed the REF** at (595.5, 41.5)
- removed the REF** at (602.5, 40.1)
- removed the REF** at (609.4, 39.7)
- removed the REF** at (168.6, 580.5)
- removed the REF** at (616.2, 40.0)
- removed the REF** at (624.7, 41.7)
- removed the REF** at (630.7, 44.3)
- removed the REF** at (637.1, 48.8)
- removed the REF** at (644.2, 57.1)
- removed the REF** at (656.3, 83.5)
- removed the REF** at (666.8, 107.6)
- removed the REF** at (678.7, 118.8)
- removed the REF** at (685.7, 119.5)
- removed the REF** at (692.8, 115.1)
- removed the REF** at (201.1, 609.4)
- removed the REF** at (705.0, 102.8)
- removed the REF** at (717.4, 87.0)
- removed the REF** at (730.0, 70.5)
- removed the REF** at (737.7, 62.2)
- removed the REF** at (744.9, 57.1)
- removed the REF** at (75.6, 39.5)
- removed the REF** at (80.9, 82.1)
- removed the REF** at (86.6, 119.8)
- removed the REF** at (94.2, 163.4)
- removed the REF** at (102.9, 207.5)
- removed the REF** at (226.8, 650.3)
- removed the REF** at (111.8, 249.2)
- removed the REF** at (121.0, 289.1)
- removed the REF** at (130.7, 328.2)
- removed the REF** at (140.7, 366.7)
- removed the REF** at (151.7, 406.9)
- removed the REF** at (162.7, 451.6)
- removed the REF** at (167.1, 497.2)
- removed the REF** at (161.5, 540.6)
- removed the REF** at (162.5, 557.4)
- removed the REF** at (183.5, 591.8)
- removed the REF** at (218.0, 701.2)
- removed the REF** at (217.1, 621.0)
- removed the REF** at (237.4, 684.4)
- removed the REF** at (228.5, 714.0)
- removed the REF** at (58.9, 22.4)
- removed the REF** at (218.7, 727.9)
- removed the REF** at (55.4, 22.0)
- removed the REF** at (60.3, 65.4)
- removed the REF** at (66.0, 105.7)
- removed the REF** at (72.9, 146.4)
- removed the REF** at (81.3, 191.0)
- removed the REF** at (90.4, 234.1)
- removed the REF** at (99.8, 275.5)
- removed the REF** at (109.3, 314.7)
- removed the REF** at (119.1, 353.0)
- removed the REF** at (63.8, 65.7)
- removed the REF** at (130.2, 393.8)
- removed the REF** at (140.5, 434.7)
- removed the REF** at (147.2, 477.9)
- removed the REF** at (145.9, 519.5)
- removed the REF** at (146.8, 554.6)
- removed the REF** at (165.7, 582.5)
- removed the REF** at (198.2, 611.5)
- removed the REF** at (223.3, 650.6)
- removed the REF** at (215.2, 699.0)
- removed the REF** at (215.1, 728.4)
- removed the REF** at (69.6, 105.9)
- removed the REF** at (71.0, 10.7)
- removed the REF** at (229.7, 737.6)
- removed the REF** at (28.8, 28.8)
- removed the REF** at (18.5, 18.5)
- removed the REF** at (18.3, 18.3)
- removed the REF** at (72.2, 72.2)
- removed the REF** at (61.9, 61.9)
- removed the REF** at (61.7, 61.7)
- removed the REF** at (112.4, 112.4)
- removed the REF** at (102.2, 102.2)
- removed the REF** at (76.4, 146.6)
- removed the REF** at (101.9, 101.9)
- removed the REF** at (153.1, 153.1)
- removed the REF** at (143.0, 143.0)
- removed the REF** at (142.7, 142.7)
- removed the REF** at (197.6, 197.6)
- removed the REF** at (187.5, 187.5)
- removed the REF** at (187.2, 187.2)
- removed the REF** at (240.8, 240.8)
- removed the REF** at (230.7, 230.7)
- removed the REF** at (230.3, 230.3)
- removed the REF** at (84.9, 191.0)
- removed the REF** at (282.1, 282.1)
- removed the REF** at (272.1, 272.1)
- removed the REF** at (271.7, 271.7)
- removed the REF** at (321.3, 321.3)
- removed the REF** at (311.3, 311.3)
- removed the REF** at (310.9, 310.9)
- removed the REF** at (359.5, 359.5)
- removed the REF** at (349.6, 349.6)
- removed the REF** at (349.2, 349.2)
- removed the REF** at (400.3, 400.3)
- removed the REF** at (93.9, 234.1)
- removed the REF** at (390.4, 390.4)
- removed the REF** at (390.0, 390.0)
- removed the REF** at (441.3, 441.3)
- removed the REF** at (431.3, 431.3)
- removed the REF** at (430.9, 430.9)
- removed the REF** at (484.7, 484.7)
- removed the REF** at (474.3, 474.3)
- removed the REF** at (474.2, 474.2)
- removed the REF** at (526.4, 526.4)
- removed the REF** at (515.9, 515.9)
- removed the REF** at (103.3, 275.4)
- removed the REF** at (516.1, 516.1)
- removed the REF** at (561.3, 561.3)
- removed the REF** at (551.2, 551.2)
- removed the REF** at (550.8, 550.8)
- removed the REF** at (587.0, 587.0)
- removed the REF** at (580.4, 580.4)
- removed the REF** at (579.2, 579.2)
- removed the REF** at (615.8, 615.8)
- removed the REF** at (609.5, 609.5)
- removed the REF** at (608.2, 608.2)
- removed the REF** at (112.8, 314.6)
- removed the REF** at (657.1, 657.1)
- removed the REF** at (647.2, 647.2)
- removed the REF** at (646.8, 646.8)
- removed the REF** at (705.4, 705.4)
- removed the REF** at (695.5, 695.5)
- removed the REF** at (696.2, 696.2)
- removed the REF** at (734.7, 734.7)
- removed the REF** at (725.2, 725.2)
- removed the REF** at (724.6, 724.6)
- removed the REF** at (4.98, 85.3)
- added REF**: QFN-24-1EP_4x4mm_Pitch0.5mm, QFN-24-1EP_4x4mm_Pitch0.5mm, B.Cu at (122.7, -352.8)
- added REF**: CL-Z891, CL-Z891, B.Cu at (15.9, -84.9)
- added REF**: CL-Z891, CL-Z891, B.Cu at (26.7, -84.4)
- added REF**: CL-Z891, CL-Z891, B.Cu at (37.6, -83.9)
- added REF**: CL-Z891, CL-Z891, B.Cu at (48.4, -83.4)
- added REF**: CL-Z891, CL-Z891, B.Cu at (59.3, -82.9)
- added REF**: CL-Z891, CL-Z891, B.Cu at (72.2, -82.4)
- added REF**: CL-Z891, CL-Z891, B.Cu at (81.8, -82.0)
- added REF**: CL-Z891, CL-Z891, B.Cu at (91.4, -81.7)
- added REF**: CL-Z891, CL-Z891, B.Cu at (101.0, -81.4)
- added REF**: CL-Z891, CL-Z891, B.Cu at (110.6, -81.0)
- added REF**: QFN-24-1EP_4x4mm_Pitch0.5mm, QFN-24-1EP_4x4mm_Pitch0.5mm, B.Cu at (133.8, -393.6)
- added REF**: CL-Z891, CL-Z891, B.Cu at (120.1, -80.7)
- added REF**: CL-Z891, CL-Z891, B.Cu at (129.7, -80.4)
- added REF**: CL-Z891, CL-Z891, B.Cu at (142.5, -80.0)
- added REF**: CL-Z891, CL-Z891, B.Cu at (153.2, -79.7)
- added REF**: CL-Z891, CL-Z891, B.Cu at (163.9, -79.4)
- added REF**: CL-Z891, CL-Z891, B.Cu at (174.6, -79.1)
- added REF**: CL-Z891, CL-Z891, B.Cu at (185.2, -78.9)
- added REF**: CL-Z891, CL-Z891, B.Cu at (195.9, -78.6)
- added REF**: CL-Z891, CL-Z891, B.Cu at (208.6, -78.3)
- added REF**: CL-Z891, CL-Z891, B.Cu at (219.2, -78.0)
- added REF**: QFN-24-1EP_4x4mm_Pitch0.5mm, QFN-24-1EP_4x4mm_Pitch0.5mm, B.Cu at (144.1, -434.6)
- added REF**: CL-Z891, CL-Z891, B.Cu at (229.7, -77.8)
- added REF**: CL-Z891, CL-Z891, B.Cu at (240.3, -77.6)
- added REF**: CL-Z891, CL-Z891, B.Cu at (250.8, -77.3)
- added REF**: CL-Z891, CL-Z891, B.Cu at (261.3, -77.1)
- added REF**: CL-Z891, CL-Z891, B.Cu at (274.0, -76.9)
- added REF**: CL-Z891, CL-Z891, B.Cu at (282.9, -76.7)
- added REF**: CL-Z891, CL-Z891, B.Cu at (291.8, -76.5)
- added REF**: CL-Z891, CL-Z891, B.Cu at (300.7, -76.3)
- added REF**: CL-Z891, CL-Z891, B.Cu at (309.7, -76.1)
- added REF**: CL-Z891, CL-Z891, B.Cu at (318.6, -75.9)
- added REF**: QFN-24-1EP_4x4mm_Pitch0.5mm, QFN-24-1EP_4x4mm_Pitch0.5mm, B.Cu at (150.7, -478.3)
- added REF**: CL-Z891, CL-Z891, B.Cu at (331.1, -75.7)
- added REF**: CL-Z891, CL-Z891, B.Cu at (340.5, -75.5)
- added REF**: CL-Z891, CL-Z891, B.Cu at (349.8, -75.3)
- added REF**: CL-Z891, CL-Z891, B.Cu at (359.1, -75.1)
- added REF**: CL-Z891, CL-Z891, B.Cu at (368.4, -74.9)
- added REF**: CL-Z891, CL-Z891, B.Cu at (380.9, -74.7)
- added REF**: CL-Z891, CL-Z891, B.Cu at (390.6, -74.4)
- added REF**: CL-Z891, CL-Z891, B.Cu at (400.2, -74.5)
- added REF**: CL-Z891, CL-Z891, B.Cu at (409.8, -74.9)
- added REF**: CL-Z891, CL-Z891, B.Cu at (419.5, -75.4)
- added REF**: QFN-24-1EP_4x4mm_Pitch0.5mm, QFN-24-1EP_4x4mm_Pitch0.5mm, B.Cu at (149.3, -520.7)
- added REF**: CL-Z891, CL-Z891, B.Cu at (432.1, -76.5)
- added REF**: CL-Z891, CL-Z891, B.Cu at (442.0, -77.7)
- added REF**: CL-Z891, CL-Z891, B.Cu at (451.9, -79.2)
- added REF**: CL-Z891, CL-Z891, B.Cu at (461.9, -81.2)
- added REF**: CL-Z891, CL-Z891, B.Cu at (474.8, -84.3)
- added REF**: CL-Z891, CL-Z891, B.Cu at (483.4, -86.9)
- added REF**: CL-Z891, CL-Z891, B.Cu at (492.1, -89.9)
- added REF**: CL-Z891, CL-Z891, B.Cu at (500.8, -92.9)
- added REF**: CL-Z891, CL-Z891, B.Cu at (513.7, -97.5)
- added REF**: CL-Z891, CL-Z891, B.Cu at (522.5, -99.0)
- added REF**: QFN-24-1EP_4x4mm_Pitch0.5mm, QFN-24-1EP_4x4mm_Pitch0.5mm, B.Cu at (150.4, -554.6)
- added REF**: CL-Z891, CL-Z891, B.Cu at (531.3, -99.1)
- added REF**: CL-Z891, CL-Z891, B.Cu at (540.0, -99.2)
- added REF**: CL-Z891, CL-Z891, B.Cu at (552.9, -81.9)
- added REF**: CL-Z891, CL-Z891, B.Cu at (562.4, -66.3)
- added REF**: CL-Z891, CL-Z891, B.Cu at (571.0, -55.8)
- added REF**: CL-Z891, CL-Z891, B.Cu at (578.9, -49.5)
- added REF**: CL-Z891, CL-Z891, B.Cu at (588.3, -43.9)
- added REF**: CL-Z891, CL-Z891, B.Cu at (595.5, -41.5)
- added REF**: CL-Z891, CL-Z891, B.Cu at (602.5, -40.1)
- added REF**: CL-Z891, CL-Z891, B.Cu at (609.4, -39.7)
- added REF**: QFN-24-1EP_4x4mm_Pitch0.5mm, QFN-24-1EP_4x4mm_Pitch0.5mm, B.Cu at (168.6, -580.5)
- added REF**: CL-Z891, CL-Z891, B.Cu at (616.2, -40.0)
- added REF**: CL-Z891, CL-Z891, B.Cu at (624.7, -41.7)
- added REF**: CL-Z891, CL-Z891, B.Cu at (630.7, -44.3)
- added REF**: CL-Z891, CL-Z891, B.Cu at (637.1, -48.8)
- added REF**: CL-Z891, CL-Z891, B.Cu at (644.2, -57.1)
- added REF**: CL-Z891, CL-Z891, B.Cu at (656.3, -83.5)
- added REF**: CL-Z891, CL-Z891, B.Cu at (666.8, -107.6)
- added REF**: CL-Z891, CL-Z891, B.Cu at (678.7, -118.8)
- added REF**: CL-Z891, CL-Z891, B.Cu at (685.7, -119.5)
- added REF**: CL-Z891, CL-Z891, B.Cu at (692.8, -115.1)
- added REF**: QFN-24-1EP_4x4mm_Pitch0.5mm, QFN-24-1EP_4x4mm_Pitch0.5mm, B.Cu at (201.1, -609.4)
- added REF**: CL-Z891, CL-Z891, B.Cu at (705.0, -102.8)
- added REF**: CL-Z891, CL-Z891, B.Cu at (717.4, -87.0)
- added REF**: CL-Z891, CL-Z891, B.Cu at (730.0, -70.5)
- added REF**: CL-Z891, CL-Z891, B.Cu at (737.7, -62.2)
- added REF**: CL-Z891, CL-Z891, B.Cu at (744.9, -57.1)
- added REF**: cut_point, cut_point, B.Cu at (75.6, -39.5)
- added REF**: cut_point, cut_point, B.Cu at (80.9, -82.1)
- added REF**: cut_point, cut_point, B.Cu at (86.6, -119.8)
- added REF**: cut_point, cut_point, B.Cu at (94.2, -163.4)
- added REF**: cut_point, cut_point, B.Cu at (102.9, -207.5)
- added REF**: QFN-24-1EP_4x4mm_Pitch0.5mm, QFN-24-1EP_4x4mm_Pitch0.5mm, B.Cu at (226.8, -650.3)
- added REF**: cut_point, cut_point, B.Cu at (111.8, -249.2)
- added REF**: cut_point, cut_point, B.Cu at (121.0, -289.1)
- added REF**: cut_point, cut_point, B.Cu at (130.7, -328.2)
- added REF**: cut_point, cut_point, B.Cu at (140.7, -366.7)
- added REF**: cut_point, cut_point, B.Cu at (151.7, -406.9)
- added REF**: cut_point, cut_point, B.Cu at (162.7, -451.6)
- added REF**: cut_point, cut_point, B.Cu at (167.1, -497.2)
- added REF**: cut_point, cut_point, B.Cu at (161.5, -540.6)
- added REF**: cut_point, cut_point, B.Cu at (162.5, -557.4)
- added REF**: cut_point, cut_point, B.Cu at (183.5, -591.8)
- added REF**: QFN-24-1EP_4x4mm_Pitch0.5mm, QFN-24-1EP_4x4mm_Pitch0.5mm, B.Cu at (218.0, -701.2)
- added REF**: cut_point, cut_point, B.Cu at (217.1, -621.0)
- added REF**: cut_point, cut_point, B.Cu at (237.4, -684.4)
- added REF**: cut_point, cut_point, B.Cu at (228.5, -714.0)
- added REF**: QFN-24-1EP_4x4mm_Pitch0.5mm, QFN-24-1EP_4x4mm_Pitch0.5mm, B.Cu at (58.9, -22.4)
- added REF**: QFN-24-1EP_4x4mm_Pitch0.5mm, QFN-24-1EP_4x4mm_Pitch0.5mm, B.Cu at (218.7, -727.9)
- added REF**: R_0402, R_0402, B.Cu at (55.4, -22.0)
- added REF**: R_0402, R_0402, B.Cu at (60.3, -65.4)
- added REF**: R_0402, R_0402, B.Cu at (66.0, -105.7)
- added REF**: R_0402, R_0402, B.Cu at (72.9, -146.4)
- added REF**: R_0402, R_0402, B.Cu at (81.3, -191.0)
- added REF**: R_0402, R_0402, B.Cu at (90.4, -234.1)
- added REF**: R_0402, R_0402, B.Cu at (99.8, -275.5)
- added REF**: R_0402, R_0402, B.Cu at (109.3, -314.7)
- added REF**: R_0402, R_0402, B.Cu at (119.1, -353.0)
- added REF**: QFN-24-1EP_4x4mm_Pitch0.5mm, QFN-24-1EP_4x4mm_Pitch0.5mm, B.Cu at (63.8, -65.7)
- added REF**: R_0402, R_0402, B.Cu at (130.2, -393.8)
- added REF**: R_0402, R_0402, B.Cu at (140.5, -434.7)
- added REF**: R_0402, R_0402, B.Cu at (147.2, -477.9)
- added REF**: R_0402, R_0402, B.Cu at (145.9, -519.5)
- added REF**: R_0402, R_0402, B.Cu at (146.8, -554.6)
- added REF**: R_0402, R_0402, B.Cu at (165.7, -582.5)
- added REF**: R_0402, R_0402, B.Cu at (198.2, -611.5)
- added REF**: R_0402, R_0402, B.Cu at (223.3, -650.6)
- added REF**: R_0402, R_0402, B.Cu at (215.2, -699.0)
- added REF**: R_0402, R_0402, B.Cu at (215.1, -728.4)
- added REF**: QFN-24-1EP_4x4mm_Pitch0.5mm, QFN-24-1EP_4x4mm_Pitch0.5mm, B.Cu at (69.6, -105.9)
- added REF**: BM04B-ACHSS, BM04B-ACHSS, B.Cu at (71.0, -10.7)
- added REF**: BM04B-ACHSS, BM04B-ACHSS, B.Cu at (229.7, -737.6)
- added REF**: C_0603, C_0603, B.Cu at (28.8, -28.8)
- added REF**: C_0603, C_0603, B.Cu at (18.5, -18.5)
- added REF**: C_0603, C_0603, B.Cu at (18.3, -18.3)
- added REF**: C_0603, C_0603, B.Cu at (72.2, -72.2)
- added REF**: C_0603, C_0603, B.Cu at (61.9, -61.9)
- added REF**: C_0603, C_0603, B.Cu at (61.7, -61.7)
- added REF**: C_0603, C_0603, B.Cu at (112.4, -112.4)
- added REF**: C_0603, C_0603, B.Cu at (102.2, -102.2)
- added REF**: QFN-24-1EP_4x4mm_Pitch0.5mm, QFN-24-1EP_4x4mm_Pitch0.5mm, B.Cu at (76.4, -146.6)
- added REF**: C_0603, C_0603, B.Cu at (101.9, -101.9)
- added REF**: C_0603, C_0603, B.Cu at (153.1, -153.1)
- added REF**: C_0603, C_0603, B.Cu at (143.0, -143.0)
- added REF**: C_0603, C_0603, B.Cu at (142.7, -142.7)
- added REF**: C_0603, C_0603, B.Cu at (197.6, -197.6)
- added REF**: C_0603, C_0603, B.Cu at (187.5, -187.5)
- added REF**: C_0603, C_0603, B.Cu at (187.2, -187.2)
- added REF**: C_0603, C_0603, B.Cu at (240.8, -240.8)
- added REF**: C_0603, C_0603, B.Cu at (230.7, -230.7)
- added REF**: C_0603, C_0603, B.Cu at (230.3, -230.3)
- added REF**: QFN-24-1EP_4x4mm_Pitch0.5mm, QFN-24-1EP_4x4mm_Pitch0.5mm, B.Cu at (84.9, -191.0)
- added REF**: C_0603, C_0603, B.Cu at (282.1, -282.1)
- added REF**: C_0603, C_0603, B.Cu at (272.1, -272.1)
- added REF**: C_0603, C_0603, B.Cu at (271.7, -271.7)
- added REF**: C_0603, C_0603, B.Cu at (321.3, -321.3)
- added REF**: C_0603, C_0603, B.Cu at (311.3, -311.3)
- added REF**: C_0603, C_0603, B.Cu at (310.9, -310.9)
- added REF**: C_0603, C_0603, B.Cu at (359.5, -359.5)
- added REF**: C_0603, C_0603, B.Cu at (349.6, -349.6)
- added REF**: C_0603, C_0603, B.Cu at (349.2, -349.2)
- added REF**: C_0603, C_0603, B.Cu at (400.3, -400.3)
- added REF**: QFN-24-1EP_4x4mm_Pitch0.5mm, QFN-24-1EP_4x4mm_Pitch0.5mm, B.Cu at (93.9, -234.1)
- added REF**: C_0603, C_0603, B.Cu at (390.4, -390.4)
- added REF**: C_0603, C_0603, B.Cu at (390.0, -390.0)
- added REF**: C_0603, C_0603, B.Cu at (441.3, -441.3)
- added REF**: C_0603, C_0603, B.Cu at (431.3, -431.3)
- added REF**: C_0603, C_0603, B.Cu at (430.9, -430.9)
- added REF**: C_0603, C_0603, B.Cu at (484.7, -484.7)
- added REF**: C_0603, C_0603, B.Cu at (474.3, -474.3)
- added REF**: C_0603, C_0603, B.Cu at (474.2, -474.2)
- added REF**: C_0603, C_0603, B.Cu at (526.4, -526.4)
- added REF**: C_0603, C_0603, B.Cu at (515.9, -515.9)
- added REF**: QFN-24-1EP_4x4mm_Pitch0.5mm, QFN-24-1EP_4x4mm_Pitch0.5mm, B.Cu at (103.3, -275.4)
- added REF**: C_0603, C_0603, B.Cu at (516.1, -516.1)
- added REF**: C_0603, C_0603, B.Cu at (561.3, -561.3)
- added REF**: C_0603, C_0603, B.Cu at (551.2, -551.2)
- added REF**: C_0603, C_0603, B.Cu at (550.8, -550.8)
- added REF**: C_0603, C_0603, B.Cu at (587.0, -587.0)
- added REF**: C_0603, C_0603, B.Cu at (580.4, -580.4)
- added REF**: C_0603, C_0603, B.Cu at (579.2, -579.2)
- added REF**: C_0603, C_0603, B.Cu at (615.8, -615.8)
- added REF**: C_0603, C_0603, B.Cu at (609.5, -609.5)
- added REF**: C_0603, C_0603, B.Cu at (608.2, -608.2)
- added REF**: QFN-24-1EP_4x4mm_Pitch0.5mm, QFN-24-1EP_4x4mm_Pitch0.5mm, B.Cu at (112.8, -314.6)
- added REF**: C_0603, C_0603, B.Cu at (657.1, -657.1)
- added REF**: C_0603, C_0603, B.Cu at (647.2, -647.2)
- added REF**: C_0603, C_0603, B.Cu at (646.8, -646.8)
- added REF**: C_0603, C_0603, B.Cu at (705.4, -705.4)
- added REF**: C_0603, C_0603, B.Cu at (695.5, -695.5)
- added REF**: C_0603, C_0603, B.Cu at (696.2, -696.2)
- added REF**: C_0603, C_0603, B.Cu at (734.7, -734.7)
- added REF**: C_0603, C_0603, B.Cu at (725.2, -725.2)
- added REF**: C_0603, C_0603, B.Cu at (724.6, -724.6)
- added REF**: CL-Z891, CL-Z891, B.Cu at (4.98, -85.3)
Routing:
- net (no net): track 16691.9 -> 21472.6 mm
